File: kicad/40%ish V2.kicad_pcb (KiCad board)
At the start: 2 copper layers, 21 parts, among them SW1 SW_Push, SW1-2 SW_Push, SW2 SW_Push, SW2-2 SW_Push, SW3 SW_Push, SW3-2 SW_Push, U1 Nice_Nano_V2, U3 XIAO-RP2040-DIP

Commit message: add new schematic
Parts:
- added REF**: SolderJumper-2_P1.3mm_Open_TrianglePad1.0x1.5mm, Jumper:SolderJumper-2_P1.3mm_Open_TrianglePad1.0x1.5mm, F.Cu at (107.5, 47.0)
- added REF**: SolderJumper-2_P1.3mm_Open_TrianglePad1.0x1.5mm, Jumper:SolderJumper-2_P1.3mm_Open_TrianglePad1.0x1.5mm, F.Cu at (100.0, 43.7)
- added REF**: SolderJumper-2_P1.3mm_Open_TrianglePad1.0x1.5mm, Jumper:SolderJumper-2_P1.3mm_Open_TrianglePad1.0x1.5mm, F.Cu at (97.5, 43.7)
- added REF**: SolderJumper-2_P1.3mm_Open_TrianglePad1.0x1.5mm, Jumper:SolderJumper-2_P1.3mm_Open_TrianglePad1.0x1.5mm, F.Cu at (51.5, 50.0)
- added REF**: SolderJumper-2_P1.3mm_Open_TrianglePad1.0x1.5mm, Jumper:SolderJumper-2_P1.3mm_Open_TrianglePad1.0x1.5mm, F.Cu at (51.5, 47.5)
- added REF**: SolderJumper-2_P1.3mm_Open_TrianglePad1.0x1.5mm, Jumper:SolderJumper-2_P1.3mm_Open_TrianglePad1.0x1.5mm, F.Cu at (51.5, 24.8)
- added REF**: SolderJumper-2_P1.3mm_Open_TrianglePad1.0x1.5mm, Jumper:SolderJumper-2_P1.3mm_Open_TrianglePad1.0x1.5mm, F.Cu at (100.0, 47.0)
- added REF**: SolderJumper-2_P1.3mm_Open_TrianglePad1.0x1.5mm, Jumper:SolderJumper-2_P1.3mm_Open_TrianglePad1.0x1.5mm, F.Cu at (97.5, 50.3)
- added REF**: SolderJumper-2_P1.3mm_Open_TrianglePad1.0x1.5mm, Jumper:SolderJumper-2_P1.3mm_Open_TrianglePad1.0x1.5mm, F.Cu at (60.5, 32.5)
- added REF**: SolderJumper-2_P1.3mm_Open_TrianglePad1.0x1.5mm, Jumper:SolderJumper-2_P1.3mm_Open_TrianglePad1.0x1.5mm, F.Cu at (105.0, 50.3)
- added REF**: SolderJumper-2_P1.3mm_Open_TrianglePad1.0x1.5mm, Jumper:SolderJumper-2_P1.3mm_Open_TrianglePad1.0x1.5mm, F.Cu at (51.5, 22.2)
- added REF**: SolderJumper-2_P1.3mm_Open_TrianglePad1.0x1.5mm, Jumper:SolderJumper-2_P1.3mm_Open_TrianglePad1.0x1.5mm, F.Cu at (60.5, 40.0)
- added REF**: SolderJumper-2_P1.3mm_Open_TrianglePad1.0x1.5mm, Jumper:SolderJumper-2_P1.3mm_Open_TrianglePad1.0x1.5mm, F.Cu at (60.5, 42.5)
- added REF**: SolderJumper-2_P1.3mm_Open_TrianglePad1.0x1.5mm, Jumper:SolderJumper-2_P1.3mm_Open_TrianglePad1.0x1.5mm, F.Cu at (100.0, 53.6)
- added REF**: SolderJumper-2_P1.3mm_Open_TrianglePad1.0x1.5mm, Jumper:SolderJumper-2_P1.3mm_Open_TrianglePad1.0x1.5mm, F.Cu at (100.0, 50.3)
- added REF**: SolderJumper-2_P1.3mm_Open_TrianglePad1.0x1.5mm, Jumper:SolderJumper-2_P1.3mm_Open_TrianglePad1.0x1.5mm, F.Cu at (107.5, 53.6)
- added REF**: SolderJumper-2_P1.3mm_Open_TrianglePad1.0x1.5mm, Jumper:SolderJumper-2_P1.3mm_Open_TrianglePad1.0x1.5mm, F.Cu at (105.0, 53.6)
- added REF**: SolderJumper-2_P1.3mm_Open_TrianglePad1.0x1.5mm, Jumper:SolderJumper-2_P1.3mm_Open_TrianglePad1.0x1.5mm, F.Cu at (105.0, 43.7)
- added REF**: SolderJumper-2_P1.3mm_Open_TrianglePad1.0x1.5mm, Jumper:SolderJumper-2_P1.3mm_Open_TrianglePad1.0x1.5mm, F.Cu at (60.5, 50.0)
- added REF**: SolderJumper-2_P1.3mm_Open_TrianglePad1.0x1.5mm, Jumper:SolderJumper-2_P1.3mm_Open_TrianglePad1.0x1.5mm, F.Cu at (97.5, 53.6)
- added REF**: SolderJumper-2_P1.3mm_Open_TrianglePad1.0x1.5mm, Jumper:SolderJumper-2_P1.3mm_Open_TrianglePad1.0x1.5mm, F.Cu at (105.0, 47.0)
- added REF**: SolderJumper-2_P1.3mm_Open_TrianglePad1.0x1.5mm, Jumper:SolderJumper-2_P1.3mm_Open_TrianglePad1.0x1.5mm, F.Cu at (60.5, 47.5)
- added REF**: SolderJumper-2_P1.3mm_Open_TrianglePad1.0x1.5mm, Jumper:SolderJumper-2_P1.3mm_Open_TrianglePad1.0x1.5mm, F.Cu at (102.5, 53.6)
- added REF**: SolderJumper-2_P1.3mm_Open_TrianglePad1.0x1.5mm, Jumper:SolderJumper-2_P1.3mm_Open_TrianglePad1.0x1.5mm, F.Cu at (51.5, 42.2)
- added REF**: SolderJumper-2_P1.3mm_Open_TrianglePad1.0x1.5mm, Jumper:SolderJumper-2_P1.3mm_Open_TrianglePad1.0x1.5mm, F.Cu at (51.5, 32.2)
- added REF**: SolderJumper-2_P1.3mm_Open_TrianglePad1.0x1.5mm, Jumper:SolderJumper-2_P1.3mm_Open_TrianglePad1.0x1.5mm, F.Cu at (107.5, 50.3)
- added REF**: SolderJumper-2_P1.3mm_Open_TrianglePad1.0x1.5mm, Jumper:SolderJumper-2_P1.3mm_Open_TrianglePad1.0x1.5mm, F.Cu at (51.5, 34.8)
- added REF**: SolderJumper-2_P1.3mm_Open_TrianglePad1.0x1.5mm, Jumper:SolderJumper-2_P1.3mm_Open_TrianglePad1.0x1.5mm, B.Cu at (118.8, 61.1)
- added REF**: SolderJumper-2_P1.3mm_Open_TrianglePad1.0x1.5mm, Jumper:SolderJumper-2_P1.3mm_Open_TrianglePad1.0x1.5mm, B.Cu at (121.2, 61.1)
- added REF**: SolderJumper-2_P1.3mm_Open_TrianglePad1.0x1.5mm, Jumper:SolderJumper-2_P1.3mm_Open_TrianglePad1.0x1.5mm, B.Cu at (121.2, 54.5)
- added REF**: SolderJumper-2_P1.3mm_Open_TrianglePad1.0x1.5mm, Jumper:SolderJumper-2_P1.3mm_Open_TrianglePad1.0x1.5mm, B.Cu at (118.8, 51.2)
- added REF**: SolderJumper-2_P1.3mm_Open_TrianglePad1.0x1.5mm, Jumper:SolderJumper-2_P1.3mm_Open_TrianglePad1.0x1.5mm, B.Cu at (121.2, 51.2)
- added REF**: SolderJumper-2_P1.3mm_Open_TrianglePad1.0x1.5mm, Jumper:SolderJumper-2_P1.3mm_Open_TrianglePad1.0x1.5mm, F.Cu at (60.5, 37.5)
- added REF**: SolderJumper-2_P1.3mm_Open_TrianglePad1.0x1.5mm, Jumper:SolderJumper-2_P1.3mm_Open_TrianglePad1.0x1.5mm, B.Cu at (88.8, 54.5)
- added REF**: SolderJumper-2_P1.3mm_Open_TrianglePad1.0x1.5mm, Jumper:SolderJumper-2_P1.3mm_Open_TrianglePad1.0x1.5mm, B.Cu at (113.8, 57.8)
- added REF**: SolderJumper-2_P1.3mm_Open_TrianglePad1.0x1.5mm, Jumper:SolderJumper-2_P1.3mm_Open_TrianglePad1.0x1.5mm, B.Cu at (118.8, 54.5)
- added REF**: SolderJumper-2_P1.3mm_Open_TrianglePad1.0x1.5mm, Jumper:SolderJumper-2_P1.3mm_Open_TrianglePad1.0x1.5mm, B.Cu at (113.8, 61.1)
- added REF**: SolderJumper-2_P1.3mm_Open_TrianglePad1.0x1.5mm, Jumper:SolderJumper-2_P1.3mm_Open_TrianglePad1.0x1.5mm, B.Cu at (113.8, 54.5)
- added REF**: SolderJumper-2_P1.3mm_Open_TrianglePad1.0x1.5mm, Jumper:SolderJumper-2_P1.3mm_Open_TrianglePad1.0x1.5mm, B.Cu at (118.8, 57.8)
- added REF**: SolderJumper-2_P1.3mm_Open_TrianglePad1.0x1.5mm, Jumper:SolderJumper-2_P1.3mm_Open_TrianglePad1.0x1.5mm, B.Cu at (113.8, 51.2)
- added REF**: SolderJumper-2_P1.3mm_Open_TrianglePad1.0x1.5mm, Jumper:SolderJumper-2_P1.3mm_Open_TrianglePad1.0x1.5mm, B.Cu at (116.2, 61.1)
- added REF**: SolderJumper-2_P1.3mm_Open_TrianglePad1.0x1.5mm, Jumper:SolderJumper-2_P1.3mm_Open_TrianglePad1.0x1.5mm, B.Cu at (111.2, 51.2)
- added REF**: SolderJumper-2_P1.3mm_Open_TrianglePad1.0x1.5mm, Jumper:SolderJumper-2_P1.3mm_Open_TrianglePad1.0x1.5mm, B.Cu at (111.2, 57.8)
- added REF**: SolderJumper-2_P1.3mm_Open_TrianglePad1.0x1.5mm, Jumper:SolderJumper-2_P1.3mm_Open_TrianglePad1.0x1.5mm, F.Cu at (97.5, 47.0)
- added REF**: SolderJumper-2_P1.3mm_Open_TrianglePad1.0x1.5mm, Jumper:SolderJumper-2_P1.3mm_Open_TrianglePad1.0x1.5mm, B.Cu at (121.2, 57.8)
- added REF**: SolderJumper-2_P1.3mm_Open_TrianglePad1.0x1.5mm, Jumper:SolderJumper-2_P1.3mm_Open_TrianglePad1.0x1.5mm, B.Cu at (111.2, 54.5)
- added REF**: SolderJumper-2_P1.3mm_Open_TrianglePad1.0x1.5mm, Jumper:SolderJumper-2_P1.3mm_Open_TrianglePad1.0x1.5mm, F.Cu at (51.5, 39.8)
- added REF**: SolderJumper-2_P1.3mm_Open_TrianglePad1.0x1.5mm, Jumper:SolderJumper-2_P1.3mm_Open_TrianglePad1.0x1.5mm, F.Cu at (60.5, 35.0)
- added REF**: SolderJumper-2_P1.3mm_Open_TrianglePad1.0x1.5mm, Jumper:SolderJumper-2_P1.3mm_Open_TrianglePad1.0x1.5mm, F.Cu at (51.5, 37.2)
- added REF**: SolderJumper-2_P1.3mm_Open_TrianglePad1.0x1.5mm, Jumper:SolderJumper-2_P1.3mm_Open_TrianglePad1.0x1.5mm, F.Cu at (107.5, 43.7)
- moved REF** 74.9 mm to (102.5, 34.0)
- moved U1 0.25 mm to (56.0, 35.9)
Routing:
- net unconnected-(U1-Pad1): track 0.00 -> 2.42 mm
- net unconnected-(U1-0-Pad2): track 0.00 -> 2.40 mm

Commit message: add new files and journal
Parts:
- removed REF** (x50): SolderJumper-2_P1.3mm_Open_TrianglePad1.0x1.5mm, Jumper:SolderJumper-2_P1.3mm_Open_TrianglePad1.0x1.5mm
- removed REF**: XIAO-nRF52840-Plus-SMD, Seeed Studio XIAO Series Library:XIAO-nRF52840-Plus-SMD
- removed U3: XIAO-RP2040-DIP, Seeed Studio XIAO Series Library:XIAO-RP2040-DIP
- added JP13: SolderJumper_2_Open, Jumper:SolderJumper-2_P1.3mm_Open_TrianglePad1.0x1.5mm, B.Cu at (232.9, 49.1)
- added JP14: SolderJumper_2_Open, Jumper:SolderJumper-2_P1.3mm_Open_TrianglePad1.0x1.5mm, F.Cu at (232.9, 49.1)
- added JP15: SolderJumper_2_Open, Jumper:SolderJumper-2_P1.3mm_Open_TrianglePad1.0x1.5mm, B.Cu at (241.6, 49.1)
- added JP16: SolderJumper_2_Open, Jumper:SolderJumper-2_P1.3mm_Open_TrianglePad1.0x1.5mm, F.Cu at (241.6, 49.1)
- added JP17: SolderJumper_2_Open, Jumper:SolderJumper-2_P1.3mm_Open_TrianglePad1.0x1.5mm, B.Cu at (232.9, 51.6)
- added JP18: SolderJumper_2_Open, Jumper:SolderJumper-2_P1.3mm_Open_TrianglePad1.0x1.5mm, F.Cu at (232.9, 51.6)
- added JP19: SolderJumper_2_Open, Jumper:SolderJumper-2_P1.3mm_Open_TrianglePad1.0x1.5mm, B.Cu at (241.6, 51.6)
- added JP20: SolderJumper_2_Open, Jumper:SolderJumper-2_P1.3mm_Open_TrianglePad1.0x1.5mm, F.Cu at (241.6, 51.6)
- added JP21: SolderJumper_2_Open, Jumper:SolderJumper-2_P1.3mm_Open_TrianglePad1.0x1.5mm, B.Cu at (232.9, 54.1)
- added JP22: SolderJumper_2_Open, Jumper:SolderJumper-2_P1.3mm_Open_TrianglePad1.0x1.5mm, F.Cu at (232.9, 54.1)
- added JP23: SolderJumper_2_Open, Jumper:SolderJumper-2_P1.3mm_Open_TrianglePad1.0x1.5mm, B.Cu at (241.6, 54.1)
- added JP24: SolderJumper_2_Open, Jumper:SolderJumper-2_P1.3mm_Open_TrianglePad1.0x1.5mm, F.Cu at (241.6, 54.1)
- added JP25: SolderJumper_2_Open, Jumper:SolderJumper-2_P1.3mm_Open_TrianglePad1.0x1.5mm, B.Cu at (232.9, 56.6)
- added JP26: SolderJumper_2_Open, Jumper:SolderJumper-2_P1.3mm_Open_TrianglePad1.0x1.5mm, F.Cu at (232.9, 56.6)
- added JP27: SolderJumper_2_Open, Jumper:SolderJumper-2_P1.3mm_Open_TrianglePad1.0x1.5mm, B.Cu at (241.6, 56.6)
- added JP28: SolderJumper_2_Open, Jumper:SolderJumper-2_P1.3mm_Open_TrianglePad1.0x1.5mm, F.Cu at (241.6, 56.6)
- added JP29: SolderJumper_2_Open, Jumper:SolderJumper-2_P1.3mm_Open_TrianglePad1.0x1.5mm, B.Cu at (232.9, 69.1)
- added JP30: SolderJumper_2_Open, Jumper:SolderJumper-2_P1.3mm_Open_TrianglePad1.0x1.5mm, F.Cu at (232.9, 69.1)
- added JP31: SolderJumper_2_Open, Jumper:SolderJumper-2_P1.3mm_Open_TrianglePad1.0x1.5mm, B.Cu at (234.3, 86.9)
- added JP32: SolderJumper_2_Open, Jumper:SolderJumper-2_P1.3mm_Open_TrianglePad1.0x1.5mm, F.Cu at (234.3, 86.9)
- added JP33: SolderJumper_2_Open, Jumper:SolderJumper-2_P1.3mm_Open_TrianglePad1.0x1.5mm, B.Cu at (232.9, 74.6)
- added JP34: SolderJumper_2_Open, Jumper:SolderJumper-2_P1.3mm_Open_TrianglePad1.0x1.5mm, F.Cu at (232.9, 74.6)
- added JP35: SolderJumper_2_Open, Jumper:SolderJumper-2_P1.3mm_Open_TrianglePad1.0x1.5mm, B.Cu at (232.9, 77.1)
- added JP36: SolderJumper_2_Open, Jumper:SolderJumper-2_P1.3mm_Open_TrianglePad1.0x1.5mm, F.Cu at (232.9, 77.1)
- added JP37: SolderJumper_2_Open, Jumper:SolderJumper-2_P1.3mm_Open_TrianglePad1.0x1.5mm, B.Cu at (241.6, 64.1)
- added JP38: SolderJumper_2_Open, Jumper:SolderJumper-2_P1.3mm_Open_TrianglePad1.0x1.5mm, F.Cu at (241.6, 64.1)
- added JP39: SolderJumper_2_Open, Jumper:SolderJumper-2_P1.3mm_Open_TrianglePad1.0x1.5mm, B.Cu at (241.6, 66.6)
- added JP40: SolderJumper_2_Open, Jumper:SolderJumper-2_P1.3mm_Open_TrianglePad1.0x1.5mm, F.Cu at (241.6, 66.6)
- added JP41: SolderJumper_2_Open, Jumper:SolderJumper-2_P1.3mm_Open_TrianglePad1.0x1.5mm, B.Cu at (241.6, 69.1)
- added JP42: SolderJumper_2_Open, Jumper:SolderJumper-2_P1.3mm_Open_TrianglePad1.0x1.5mm, F.Cu at (241.6, 69.1)
- added JP43: SolderJumper_2_Open, Jumper:SolderJumper-2_P1.3mm_Open_TrianglePad1.0x1.5mm, B.Cu at (238.8, 86.9)
- added JP44: SolderJumper_2_Open, Jumper:SolderJumper-2_P1.3mm_Open_TrianglePad1.0x1.5mm, F.Cu at (238.8, 86.9)
- added JP45: SolderJumper_2_Open, Jumper:SolderJumper-2_P1.3mm_Open_TrianglePad1.0x1.5mm, B.Cu at (241.6, 74.6)
- added JP46: SolderJumper_2_Open, Jumper:SolderJumper-2_P1.3mm_Open_TrianglePad1.0x1.5mm, F.Cu at (241.6, 74.6)
- added JP47: SolderJumper_2_Open, Jumper:SolderJumper-2_P1.3mm_Open_TrianglePad1.0x1.5mm, B.Cu at (241.6, 77.1)
- added JP48: SolderJumper_2_Open, Jumper:SolderJumper-2_P1.3mm_Open_TrianglePad1.0x1.5mm, F.Cu at (241.6, 77.1)
- added SW10: SW_Push, MX_Hotswap:MX-Hotswap-1U, F.Cu at (141.8, 76.1)
- added SW10-2: SW_Push, MX_Hotswap:MX-Hotswap-1U, B.Cu at (141.8, 76.1)
- added SW11: SW_Push, MX_Hotswap:MX-Hotswap-1U, F.Cu at (65.6, 97.5)
- added SW11-2: SW_Push, MX_Hotswap:MX-Hotswap-1U, B.Cu at (65.6, 97.5)
- added SW12: SW_Push, MX_Hotswap:MX-Hotswap-1U, F.Cu at (84.6, 92.8)
- added SW12-2: SW_Push, MX_Hotswap:MX-Hotswap-1U, B.Cu at (84.6, 92.8)
- added SW13: SW_Push, MX_Hotswap:MX-Hotswap-1U, F.Cu at (103.7, 90.4)
- added SW13-2: SW_Push, MX_Hotswap:MX-Hotswap-1U, B.Cu at (103.7, 90.4)
- added SW14: SW_Push, MX_Hotswap:MX-Hotswap-1U, F.Cu at (122.7, 92.8)
- added SW14-2: SW_Push, MX_Hotswap:MX-Hotswap-1U, B.Cu at (122.7, 92.8)
- added SW15: SW_Push, MX_Hotswap:MX-Hotswap-1U, F.Cu at (141.8, 95.2)
- added SW15-2: SW_Push, MX_Hotswap:MX-Hotswap-1U, B.Cu at (141.8, 95.2)
- added SW16: SW_Push, MX_Hotswap:MX-Hotswap-1U, F.Cu at (110.8, 114.2)
- added SW16-2: SW_Push, MX_Hotswap:MX-Hotswap-1U, B.Cu at (110.8, 114.2)
- added SW17: SW_Push, MX_Hotswap:MX-Hotswap-1U, F.Cu at (132.2, 116.6)
- added SW17-2: SW_Push, MX_Hotswap:MX-Hotswap-1U, B.Cu at (132.2, 116.6)
- added SW18: SW_Push, MX_Hotswap:MX-Hotswap-1.5U, F.Cu at (155.0, 121.1)
- added SW18-2: SW_Push, MX_Hotswap:MX-Hotswap-1.5U, B.Cu at (155.0, 121.1)
- added SW19: RotaryEncoder_Switch, Rotary_Encoder:RotaryEncoder_Alps_EC11E-Switch_Vertical_H20mm_CircularMountingHoles, F.Cu at (233.0, 126.9)
- added SW20: SW_Push, MX_Hotswap:MX-Hotswap-1U, F.Cu at (235.5, 119.4)
- added SW20-2: SW_Push, MX_Hotswap:MX-Hotswap-1U, B.Cu at (235.5, 119.4)
- added SW4: SW_Push, MX_Hotswap:MX-Hotswap-1U, F.Cu at (122.7, 54.7)
- added SW4-2: SW_Push, MX_Hotswap:MX-Hotswap-1U, B.Cu at (122.7, 54.7)
- added SW5: SW_Push, MX_Hotswap:MX-Hotswap-1U, F.Cu at (141.8, 57.1)
- added SW5-2: SW_Push, MX_Hotswap:MX-Hotswap-1U, B.Cu at (141.8, 57.1)
- added SW6: SW_Push, MX_Hotswap:MX-Hotswap-1U, F.Cu at (65.6, 78.5)
- added SW6-2: SW_Push, MX_Hotswap:MX-Hotswap-1U, B.Cu at (65.6, 78.5)
- added SW7: SW_Push, MX_Hotswap:MX-Hotswap-1U, F.Cu at (84.6, 73.7)
- added SW7-2: SW_Push, MX_Hotswap:MX-Hotswap-1U, B.Cu at (84.6, 73.7)
- added SW8: SW_Push, MX_Hotswap:MX-Hotswap-1U, F.Cu at (103.7, 71.3)
- added SW8-2: SW_Push, MX_Hotswap:MX-Hotswap-1U, B.Cu at (103.7, 71.3)
- added SW9: SW_Push, MX_Hotswap:MX-Hotswap-1U, F.Cu at (122.7, 73.7)
- added SW9-2: SW_Push, MX_Hotswap:MX-Hotswap-1U, B.Cu at (122.7, 73.7)
- JP1, JP11, JP3, JP5, JP7, JP9: moved to B.Cu
- JP10, JP12, JP2, JP4, JP6, JP8: moved to F.Cu
- moved U1 183.3 mm to (237.3, 62.8)
- moved SW3 122.5 mm to (103.7, 52.3)
- moved SW3-2 122.5 mm to (103.7, 52.3)
- moved SW2 121.5 mm to (84.6, 54.7)
- moved SW2-2 121.5 mm to (84.6, 54.7)
- moved SW1 119.6 mm to (65.6, 59.4)
- moved SW1-2 119.6 mm to (65.6, 59.4)
- moved JP5 40.8 mm to (241.6, 59.1), turned to 0 degrees
- moved JP6 40.8 mm to (241.6, 59.1), turned to 0 degrees
- moved JP7 37.5 mm to (241.6, 61.6)
- moved JP8 37.5 mm to (241.6, 61.6)
- moved JP2 37.4 mm to (232.9, 59.1)
- moved JP1 37.4 mm to (232.9, 59.1)
- moved JP9 37.4 mm to (232.9, 64.1)
- moved JP10 37.4 mm to (232.9, 64.1)
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Connections:
- JP1 pad 1: /VBUS -> /D21
- JP1 pad 2: Net-(JP1-B) -> /5
- JP10 pad 1: /GPIO28 -> /D4
- JP10 pad 2: Net-(JP10-B) -> /7
- JP11 pad 1: /GPIO28 -> /D18
- JP11 pad 2: Net-(JP11-B) -> /8
- JP12 pad 1: /3V3 -> /D5
- JP12 pad 2: Net-(JP11-B) -> /8
- JP2 pad 1: /GPIO26 -> /D2
- JP2 pad 2: Net-(JP1-B) -> /5
- JP3 pad 1: /GPIO26 -> /D20
- JP3 pad 2: Net-(JP3-B) -> /6
- JP4 pad 1: /VBUS -> /D3
- JP4 pad 2: Net-(JP3-B) -> /6
- JP5 pad 1: GND -> /D2
- JP5 pad 2: Net-(JP5-B) -> /20
- JP6 pad 1: /GPIO27 -> /D21
- JP6 pad 2: Net-(JP5-B) -> /20
- JP7 pad 1: /GPIO27 -> /D3
- JP7 pad 2: Net-(JP7-B) -> /19
- JP8 pad 1: GND -> /D20
- JP8 pad 2: Net-(JP7-B) -> /19
- JP9 pad 1: /3V3 -> /D19
- JP9 pad 2: Net-(JP10-B) -> /7
- SW1 pad 2: /GPIO26 -> /D1
- SW1-2 pad 2: /GPIO26 -> /D1
- SW2 pad 2: /GPIO27 -> /D0
- SW2-2 pad 2: /GPIO27 -> /D0
- SW3 pad 2: /GPIO28 -> /D2
- SW3-2 pad 2: /GPIO28 -> /D2
- U1 pad 1: unconnected-(U1-Pad1) -> /1
- U1 pad 10: unconnected-(U1-7-Pad10) -> /10
- U1 pad 11: unconnected-(U1-8-Pad11) -> /11
- U1 pad 12: unconnected-(U1-9-Pad12) -> /12
- U1 pad 13: unconnected-(U1-10-Pad13) -> /13
- U1 pad 14: unconnected-(U1-16-Pad14) -> /14
- U1 pad 15: unconnected-(U1-14-Pad15) -> /15
- U1 pad 16: unconnected-(U1-15-Pad16) -> /16
- U1 pad 17: unconnected-(U1-18-Pad17) -> /17
- U1 pad 18: unconnected-(U1-19-Pad18) -> /18
- U1 pad 19: unconnected-(U1-20-Pad19) -> /19
- U1 pad 2: unconnected-(U1-0-Pad2) -> /2
- U1 pad 20: unconnected-(U1-21-Pad20) -> /20
- U1 pad 21: unconnected-(U1-3.3v-Pad21) -> /21
- U1 pad 22: unconnected-(U1-RST-Pad22) -> /22
- U1 pad 23: unconnected-(U1-GND-Pad23) -> /23
- U1 pad 24: unconnected-(U1-B+-Pad24) -> /24
- U1 pad 25: unconnected-(U1-1-Pad25) -> /25
- U1 pad 26: unconnected-(U1-2-Pad26) -> /26
- U1 pad 27: unconnected-(U1-7-Pad27) -> /27
- U1 pad 3: unconnected-(U1-GND-Pad3) -> /3
- U1 pad 4: unconnected-(U1-GND-Pad4) -> /4
- U1 pad 5: unconnected-(U1-2-Pad5) -> /5
- U1 pad 6: unconnected-(U1-3-Pad6) -> /6
- U1 pad 7: unconnected-(U1-4-Pad7) -> /7
- U1 pad 8: unconnected-(U1-5-Pad8) -> /8
- U1 pad 9: unconnected-(U1-6-Pad9) -> /9
Routing:
- net /GPIO28: track 21.4 -> 0.00 mm, vias 2 -> 0
- net /GPIO27: track 21.4 -> 0.00 mm, vias 2 -> 0
- net /GPIO26: track 21.4 -> 0.00 mm, vias 2 -> 0
- net GND: track 8.05 -> 23.6 mm, vias 1 -> 3
- net /25: track 0.00 -> 11.5 mm
- net /VBUS: track 8.05 -> 0.00 mm, vias 1 -> 0
- net /3V3: track 8.05 -> 0.00 mm, vias 1 -> 0
- net /B+: track 0.00 -> 7.92 mm, vias 0 -> 1
- net /D2: track 0.00 -> 7.85 mm, vias 0 -> 1
- net /D20: track 0.00 -> 7.84 mm, vias 0 -> 1
- net /D21: track 0.00 -> 7.84 mm, vias 0 -> 1
- net /D19: track 0.00 -> 7.84 mm, vias 0 -> 1
- net /RST: track 0.00 -> 7.84 mm, vias 0 -> 1
- net /D6: track 0.00 -> 7.84 mm, vias 0 -> 1
- net +3V3: track 0.00 -> 7.84 mm, vias 0 -> 1
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Other:
- board outline added: 115.5 x 95.5 mm

Commit message: update PCB
Parts:
- added H1: MountingHole, MountingHole:MountingHole_3.2mm_M3, F.Cu at (75.4, 64.4)
- added H2: MountingHole, MountingHole:MountingHole_3.2mm_M3, F.Cu at (75.4, 83.2)
- added H3: MountingHole, MountingHole:MountingHole_3.2mm_M3, F.Cu at (132.0, 64.8)
- added H4: MountingHole, MountingHole:MountingHole_3.2mm_M3, F.Cu at (147.2, 108.4)
- moved SW19 78.0 mm to (159.3, 101.7)
- moved SW20 78.0 mm to (161.8, 94.2)
- moved SW20-2 78.0 mm to (161.8, 94.2)
- moved JP1 75.9 mm to (157.2, 64.7)
- moved JP10 75.9 mm to (157.2, 69.7)
- moved JP11 75.9 mm to (157.2, 72.2)
- moved JP12 75.9 mm to (157.2, 72.2)
- moved JP13 75.9 mm to (157.2, 54.7)
- moved JP14 75.9 mm to (157.2, 54.7)
- moved JP15 75.9 mm to (166.0, 54.7)
- moved JP16 75.9 mm to (166.0, 54.7)
- moved JP17 75.9 mm to (157.2, 57.2)
- moved JP18 75.9 mm to (157.2, 57.2)
- moved JP19 75.9 mm to (166.0, 57.2)
- moved JP2 75.9 mm to (157.2, 64.7)
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Routing:
- net /27: track 0.00 -> 25.6 mm
- net /D18: track 7.84 -> 21.2 mm, vias 1 -> 2
- net /D16: track 7.84 -> 21.2 mm, vias 1 -> 2
- net /D15: track 7.84 -> 21.2 mm, vias 1 -> 2
- net /D19: track 7.84 -> 21.2 mm, vias 1 -> 2
- net /D10: track 7.84 -> 21.2 mm, vias 1 -> 2
- net /D7: track 0.00 -> 13.4 mm, vias 0 -> 1
- net /D14: track 0.00 -> 13.4 mm, vias 0 -> 1
- net /D4: track 7.84 -> 21.2 mm, vias 1 -> 2
- net /D0: track 7.84 -> 21.2 mm, vias 1 -> 2
- net /D6: track 7.84 -> 21.2 mm, vias 1 -> 2
- net /D3: track 7.84 -> 21.2 mm, vias 1 -> 2
- net /D2: track 7.85 -> 21.2 mm, vias 1 -> 2
- net /D8: track 7.84 -> 21.2 mm, vias 1 -> 2
- net /D5: track 7.84 -> 21.2 mm, vias 1 -> 2
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Other:
- board text added: "3V3"
- board text added: "B+"
- board text added: "D0"
- board text added: "D1"
- board text added: "D10"
- board text added: "D15"
- board text added: "D16"
- board text added: "D18"
- board text added: "D19"
- board text added: "D2"
- board text added: "D20"
- board text added: "D21"
- board text added: "D3"
- board text added: "D4"
- board text added: "D5"
- board text added: "D6"
- board text added: "D8"
- board text added: "D9"
- board text added: "GND"
- board text added: "RST"

Commit message: PCB done
Parts:
- removed JP31, JP32, JP43, JP44: SolderJumper_2_Open, Jumper:SolderJumper-2_P1.3mm_Open_TrianglePad1.0x1.5mm
- removed SW19: RotaryEncoder_Switch, Rotary_Encoder:RotaryEncoder_Alps_EC11E-Switch_Vertical_H20mm_CircularMountingHoles
- removed SW20, SW20-2: SW_Push, MX_Hotswap:MX-Hotswap-1U
- moved SW7 0.18 mm to (84.8, 73.8)
- moved SW7-2 0.18 mm to (84.8, 73.8)
- moved JP45 0.18 mm to (166.2, 80.2)
- moved H3 0.18 mm to (132.1, 64.8)
- moved JP19 0.18 mm to (166.2, 57.2)
- moved JP20 0.18 mm to (166.2, 57.2)
- moved JP47 0.18 mm to (166.2, 82.7)
- moved JP48 0.18 mm to (166.2, 82.7)
- moved SW11 0.18 mm to (65.7, 97.6)
- moved SW11-2 0.18 mm to (65.7, 97.6)
- moved H1 0.18 mm to (75.5, 64.4)
- moved JP12 0.18 mm to (157.4, 72.2)
- moved SW17 0.18 mm to (132.4, 116.7)
- moved SW17-2 0.18 mm to (132.4, 116.7)
- moved SW15 0.18 mm to (141.9, 95.2)
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Connections:
- SW10 pad 2: /D9 -> /D5
- SW10-2 pad 2: /D9 -> /D5
- SW11 pad 2: /D10 -> /D15
- SW11-2 pad 2: /D10 -> /D15
- SW12 pad 2: /D16 -> /D6
- SW12-2 pad 2: /D16 -> /D6
- SW13 pad 2: /D14 -> /D25
- SW13-2 pad 2: /D14 -> /D25
- SW14 pad 2: /D15 -> /D26
- SW14-2 pad 2: /D15 -> /D26
- SW15 pad 2: /D18 -> /D16
- SW15-2 pad 2: /D18 -> /D16
- SW16 pad 2: /D19 -> /D8
- SW16-2 pad 2: /D19 -> /D8
- SW17 pad 2: /D20 -> /D10
- SW17-2 pad 2: /D20 -> /D10
- SW18 pad 2: /D21 -> /D9
- SW18-2 pad 2: /D21 -> /D9
- SW3 pad 2: /D2 -> /D21
- SW3-2 pad 2: /D2 -> /D21
- SW4 pad 2: /D3 -> /D2
- SW4-2 pad 2: /D3 -> /D2
- SW5 pad 2: /D4 -> /D20
- SW5-2 pad 2: /D4 -> /D20
- SW6 pad 2: /D5 -> /D3
- SW6-2 pad 2: /D5 -> /D3
- SW7 pad 2: /D6 -> /D19
- SW7-2 pad 2: /D6 -> /D19
- SW8 pad 2: /D7 -> /D4
- SW8-2 pad 2: /D7 -> /D4
- SW9 pad 2: /D8 -> /D18
- SW9-2 pad 2: /D8 -> /D18
- U1 pad 25: /25 -> /D25
- U1 pad 26: /26 -> /D26
Routing:
- net /D1: track 21.2 -> 134.6 mm, vias 2 -> 3
- net /D3: track 21.2 -> 127.9 mm, vias 2 -> 3
- net /D15: track 21.2 -> 126.6 mm
- net /D0: track 21.2 -> 113.2 mm, vias 2 -> 3
- net /D21: track 7.84 -> 96.9 mm, vias 1 -> 3
- net /D6: track 21.2 -> 104.1 mm, vias 2 -> 3
- net /D19: track 21.2 -> 103.9 mm
- net /D25: track 0.00 -> 81.2 mm, vias 0 -> 1
- net /D4: track 21.2 -> 85.0 mm, vias 2 -> 3
- net /D8: track 21.2 -> 83.4 mm, vias 2 -> 3
- net /D26: track 0.00 -> 59.2 mm, vias 0 -> 1
- net /D2: track 21.2 -> 75.8 mm, vias 2 -> 4
- net /D18: track 21.2 -> 67.4 mm
- net /D20: track 7.84 -> 52.8 mm, vias 1 -> 3
- net /D9: track 21.2 -> 61.2 mm, vias 2 -> 3
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- added copper zone on B.Cu, net GND
- added copper zone on F.Cu, net GND
