File: kicad/40%ish V2.kicad_sch (KiCad schematic)
At the start: 21 parts, among them SW1 SW_Push, SW1-2 SW_Push, SW2 SW_Push, SW2-2 SW_Push, SW3 SW_Push, SW3-2 SW_Push, U1 Nice_Nano_V2, U2 XIAO-nRF52840-DIP, U3 XIAO-RP2040-DIP

Commit message: add new schematic
Parts:
- removed U2: XIAO-nRF52840-DIP, Module:MOUDLE14P-XIAO-DIP-SMD, symbol Seeed_Studio_XIAO_Series:XIAO-nRF52840-DIP
- removed U3: XIAO-RP2040-DIP, Seeed Studio XIAO Series Library:XIAO-RP2040-DIP, symbol Seeed_Studio_XIAO_Series:XIAO-RP2040-DIP
- added JP13, JP14, JP15, JP16, JP17, JP18, JP19, JP20, JP21, JP22, JP23, JP24, JP25, JP26, JP27, JP28, JP29, JP30, JP31, JP32, JP33, JP34, JP35, JP36, JP37, JP38, JP39, JP40, JP41, JP42, JP43, JP44, JP45, JP46, JP47, JP48: SolderJumper_2_Open, Jumper:SolderJumper-2_P1.3mm_Open_TrianglePad1.0x1.5mm, symbol Jumper:SolderJumper_2_Open
- added SW10, SW10-2, SW11, SW11-2, SW12, SW12-2, SW13, SW13-2, SW14, SW14-2, SW15, SW15-2, SW16, SW16-2, SW17, SW17-2, SW18, SW18-2, SW4, SW4-2, SW5, SW5-2, SW6, SW6-2, SW7, SW7-2, SW8, SW8-2, SW9, SW9-2: SW_Push, MX_Hotswap:MX-Hotswap-1U, symbol Switch:SW_Push
Connections:
- net GND: now also JP17.1 (A), JP20.1 (A), JP22.1 (A), JP23.1 (A), JP26.1 (A), JP27.1 (A), SW10-2.1, SW10.1, SW11-2.1, SW11.1, SW12-2.1, SW12.1, SW13-2.1, SW13.1, SW14-2.1, SW14.1, SW15-2.1, SW15.1, SW16-2.1, SW16.1, SW17-2.1, SW17.1, SW18-2.1, SW18.1, SW4-2.1, SW4.1, SW5-2.1, SW5.1, SW6-2.1, SW6.1, SW7-2.1, SW7.1, SW8-2.1, SW8.1, SW9-2.1, SW9.1; no longer JP5.1 (A), JP8.1 (A)
- net 6: now reaches JP3.2 (B), JP4.2 (B)
- net 6: now also U1.6 (3)
- net 8: now reaches JP11.2 (B), JP12.2 (B)
- net 8: now also U1.8 (5)
- net 19: now reaches JP7.2 (B), JP8.2 (B)
- net 19: now also U1.19 (20)
- net 5: now reaches JP1.2 (B), JP2.2 (B)
- net 5: now also U1.5 (2)
- net 20: now reaches JP5.2 (B), JP6.2 (B)
- net 20: now also U1.20 (21)
- net 1: now reaches U1.1
- net 1: now also JP13.2 (B), JP14.2 (B)
- net 10: now reaches U1.10 (7)
- net 10: now also JP31.2 (B), JP32.2 (B)
- net 11: now reaches U1.11 (8)
- net 11: now also JP33.2 (B), JP34.2 (B)
- net 12: now reaches U1.12 (9)
- net 12: now also JP35.2 (B), JP36.2 (B)
- net 13: now reaches U1.13 (10)
- net 13: now also JP47.2 (B), JP48.2 (B)
- net 14: now reaches U1.14 (16)
- net 14: now also JP45.2 (B), JP46.2 (B)
- net 15: now reaches U1.15 (14)
- net 15: now also JP43.2 (B), JP44.2 (B)
- net 16: now reaches U1.16 (15)
- net 16: now also JP41.2 (B), JP42.2 (B)
- net 17: now reaches U1.17 (18)
- net 17: now also JP39.2 (B), JP40.2 (B)
- net 18: now reaches U1.18 (19)
- net 18: now also JP37.2 (B), JP38.2 (B)
- net 2: now reaches U1.2 (0)
- net 2: now also JP17.2 (B), JP18.2 (B)
- net 21: now reaches U1.21 (3.3v)
- net 21: now also JP27.2 (B), JP28.2 (B)
- net 22: now reaches U1.22 (RST)
- net 22: now also JP23.2 (B), JP24.2 (B)
- net 23: now reaches U1.23 (GND)
- net 23: now also JP19.2 (B), JP20.2 (B)
- net 24: now reaches U1.24 (B+)
- net 24: now also JP15.2 (B), JP16.2 (B)
- net 25: now reaches U1.25 (1)
- net 26: now reaches U1.26 (2)
- net 27: now reaches U1.27 (7)
- net 3: now reaches U1.3 (GND)
- net 3: now also JP21.2 (B), JP22.2 (B)
- net 4: now reaches U1.4 (GND)
- net 4: now also JP25.2 (B), JP26.2 (B)
- net 7: now reaches U1.7 (4)
- net 7: now also JP10.2 (B), JP9.2 (B)
- net 9: now reaches U1.9 (6)
- net 9: now also JP29.2 (B), JP30.2 (B)
- net 3V3 renamed D19
- net D19: now also JP38.1 (A); no longer JP12.1 (A)
- net GPIO26 renamed D1
- net D1: now also JP14.1 (A), JP15.1 (A); no longer JP2.1 (A), JP3.1 (A)
- net GPIO27 renamed D0
- net D0: now also JP18.1 (A), JP19.1 (A); no longer JP6.1 (A), JP7.1 (A)
- net GPIO28 renamed D2
- net D2: now also JP2.1 (A), JP5.1 (A); no longer JP10.1 (A), JP11.1 (A)
- net VBUS renamed D21
- net D21: now also JP6.1 (A); no longer JP4.1 (A)
- new net: SW18-2.2, SW18.2
- new net: SW16-2.2, SW16.2
- new net: SW14-2.2, SW14.2
- new net: SW15-2.2, SW15.2
- new net: SW13-2.2, SW13.2
- new net: SW11-2.2, SW11.2
- new net: SW12-2.2, SW12.2
- new net: SW17-2.2, SW17.2
- new net +3V3: JP25.1 (A), JP28.1 (A)
- new net B+: JP13.1 (A), JP16.1 (A)
- new net D10: JP35.1 (A), JP48.1 (A)
- new net D14: JP31.1 (A), JP44.1 (A)
- new net D15: JP29.1 (A), JP42.1 (A)
- new net D16: JP33.1 (A), JP46.1 (A)
- new net D18: JP11.1 (A), JP40.1 (A)
- new net D20: JP3.1 (A), JP8.1 (A)
- new net D3: JP4.1 (A), JP7.1 (A), SW4-2.2, SW4.2
- new net D4: JP10.1 (A), JP37.1 (A), SW5-2.2, SW5.2
- new net D5: JP12.1 (A), JP39.1 (A), SW6-2.2, SW6.2
- new net D6: JP30.1 (A), JP41.1 (A), SW7-2.2, SW7.2
- new net D7: JP32.1 (A), JP43.1 (A), SW8-2.2, SW8.2
- new net D8: JP34.1 (A), JP45.1 (A), SW9-2.2, SW9.2
- new net D9: JP36.1 (A), JP47.1 (A), SW10-2.2, SW10.2
- new net RST: JP21.1 (A), JP24.1 (A)
Other:
- moved on the sheet: SW1, SW1-2, SW2, SW2-2, SW3, SW3-2

Commit message: add new files and journal
Parts:
- added SW19: RotaryEncoder_Switch, Rotary_Encoder:RotaryEncoder_Alps_EC11E-Switch_Vertical_H20mm_CircularMountingHoles, symbol Device:RotaryEncoder_Switch
- added SW20, SW20-2: SW_Push, MX_Hotswap:MX-Hotswap-1U, symbol Switch:SW_Push
- SW18, SW18-2: footprint MX_Hotswap:MX-Hotswap-1U -> MX_Hotswap:MX-Hotswap-1.5U
Connections:
- net 25: now also SW19.B
- net 26: now also SW19.A
- net 27: now also SW19.S1, SW20-2.2, SW20.2
- net D10: now also SW11-2.2, SW11.2
- net D14: now also SW13-2.2, SW13.2
- net D15: now also SW14-2.2, SW14.2
- net D16: now also SW12-2.2, SW12.2
- net D18: now also SW15-2.2, SW15.2
- net D19: now also SW16-2.2, SW16.2
- net D20: now also SW17-2.2, SW17.2
- net D21: now also SW18-2.2, SW18.2
- net GND: now also SW19.C, SW19.S2, SW20-2.1, SW20.1

Commit message: update PCB
Parts:
- added H1, H2, H3, H4: MountingHole, MountingHole:MountingHole_3.2mm_M3, symbol Mechanical:MountingHole

Commit message: PCB done
Parts:
- removed JP31, JP32, JP43, JP44: SolderJumper_2_Open, Jumper:SolderJumper-2_P1.3mm_Open_TrianglePad1.0x1.5mm, symbol Jumper:SolderJumper_2_Open
- removed SW19: RotaryEncoder_Switch, Rotary_Encoder:RotaryEncoder_Alps_EC11E-Switch_Vertical_H20mm_CircularMountingHoles, symbol Device:RotaryEncoder_Switch
- removed SW20, SW20-2: SW_Push, MX_Hotswap:MX-Hotswap-1U, symbol Switch:SW_Push
Connections:
- net D14 is gone; now on net D25: SW13-2.2, SW13.2
- net D7 is gone; now on net D4: SW8-2.2, SW8.2
- net D10: now also SW17-2.2, SW17.2; no longer SW11-2.2, SW11.2
- net D15: now also SW11-2.2, SW11.2; no longer SW14-2.2, SW14.2
- net D16: now also SW15-2.2, SW15.2; no longer SW12-2.2, SW12.2
- net D18: now also SW9-2.2, SW9.2; no longer SW15-2.2, SW15.2
- net D19: now also SW7-2.2, SW7.2; no longer SW16-2.2, SW16.2
- net D2: now also SW4-2.2, SW4.2; no longer SW3-2.2, SW3.2
- net D20: now also SW5-2.2, SW5.2; no longer SW17-2.2, SW17.2
- net D21: now also SW3-2.2, SW3.2; no longer SW18-2.2, SW18.2
- net D3: now also SW6-2.2, SW6.2; no longer SW4-2.2, SW4.2
- net D4: no longer SW5-2.2, SW5.2
- net D5: now also SW10-2.2, SW10.2; no longer SW6-2.2, SW6.2
- net D6: now also SW12-2.2, SW12.2; no longer SW7-2.2, SW7.2
- net D8: now also SW16-2.2, SW16.2; no longer SW9-2.2, SW9.2
- net D9: now also SW18-2.2, SW18.2; no longer SW10-2.2, SW10.2
- net 25 renamed D25
- net 26 renamed D26
- net D26: now also SW14-2.2, SW14.2
Other:
- moved on the sheet: H1, H2, H3, H4

Commit message: make 3D dir
Other:
- title: (none) -> 40%ish split keyboard 
- moved on the sheet: H1, H2, H3, H4, SW1, SW1-2, SW10, SW10-2, SW11, SW11-2, SW12, SW12-2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
